Commit message: Design new basic robot

File: dev_ws/src/alpay_description/urdf/common.xacro (robot description, xacro)
@@ -5,4 +5,6 @@
     <material name="blue"> <color rgba="0 0 0.6 1"/> </material>
     <material name="gray"> <color rgba="0.6 0.6 0.6 1"/> </material>
+    <material name="light_gray"> <color rgba="0.8 0.8 0.8 1"/> </material>
+    <material name="dark_gray"> <color rgba="0.4 0.4 0.4 1"/> </material>
     <material name="black"> <color rgba="0 0 0 1"/> </material>
     <material name="white"> <color rgba="1 1 1 1"/> </material>
@@ -16,4 +18,33 @@
         </inertial>
     </xacro:macro>
+    <xacro:macro name="rect_tube_inertia" params="m t x y z xyz rpy">
+        <!-- profilin uzun kısmı için x ekseni kullanılıyor -->
+        <inertial>
+            <origin xyz="${xyz}" rpy="${rpy}"/>
+            <mass value="${m}"/>
+            <inertia ixx="${m/12*((y*z**3)-((y-2*t)*(z-2*t)**3))}"
+                     iyy="${m/12*((x*z**3)-((x-2*t)*(z-2*t)**3))}"
+                     izz="${m/12*((x*y**3)-((x-2*t)*(y-2*t)**3))}"
+                     ixy="0" ixz="0" iyz="0"/>
+        </inertial>
+    </xacro:macro>
+    <xacro:macro name="u_rect_tube_inertia" params="m t x y z xyz rpy">
+        <!-- profilin uzun kısmı için x ekseni kullanılıyor -->
+        <!-- boş olan taraf üste (+z) bakıyor -->
+        <inertial>
+            <origin xyz="${xyz}" rpy="${rpy}"/>
+            <mass value="${m}"/>
+            <inertia ixx="${m/12*(2*(y*t**3)+(y*(z-2*t)**3))}"
+                     iyy="${m/12*(2*(z*t**3)+(x*(z-2*t)**3))}"
+                     izz="${m/12*((x*y**3)-((x-2*t)*(y-2*t)**3))}"
+                     ixy="0" ixz="0" iyz="0"/>
+        </inertial>
+    </xacro:macro>
+    <xacro:macro name="structure_inertia" params="step xyz rpy">
+        <!-- structureın uzun kısmı için x ekseni kullanılıyor -->
+        <!-- boş olan taraf üste (+z) bakıyor -->
+        <xacro:u_rect_tube_inertia m="${step*0.016}" t="0.002" x="${step*0.025}"
+                                   y="0.05" z="0.05" xyz="${xyz}" rpy="${rpy}"/>
+    </xacro:macro>
     <xacro:macro name="cylinder_inertia" params="m r l xyz rpy">
         <inertial>
@@ -25,3 +56,104 @@
         </inertial>
     </xacro:macro>
+    <xacro:macro name="structure" params="link_name step xyz rpy">
+        <link name="${link_name}">
+            <collision>
+                <geometry>
+                    <box size="${step*0.05/2} 0.05 0.05"/>
+                </geometry>
+                <origin xyz="${xyz}" rpy="${rpy}"/>
+            </collision>
+            <visual>
+                <material name="white"/>
+                <geometry>
+                    <box size="${step*0.05/2} 0.05 0.05"/>
+                </geometry>
+                <origin xyz="${xyz}" rpy="${rpy}"/>
+            </visual>
+            <xacro:structure_inertia step="${step}" xyz="${xyz}" rpy="${rpy}"/>
+            <gazebo>
+                <material>Gazebo/White</material>
+            </gazebo>
+        </link>
+    </xacro:macro>
+    <xacro:macro name="traction_wheel" params="link_name xyz rpy">
+        <link name="${link_name}">
+            <visual>
+                <geometry>
+                    <cylinder radius="${wheel_diameter/2}" length="0.0375"/>
+                </geometry>
+                <material name="gray"/>
+                <origin xyz="${xyz}" rpy="${rpy}"/>
+            </visual>
+            <collision>
+                <geometry>
+                    <cylinder radius="${wheel_diameter/2}" length="0.0375"/>
+                </geometry>
+                <origin xyz="${xyz}" rpy="${rpy}"/>
+            </collision>
+            <xacro:cylinder_inertia m="0.1" r="${wheel_diameter/2}" l="0.0375" xyz="${xyz}" rpy="${rpy}"/>
+            <gazebo>
+                <material>Gazebo/Gray</material>
+                <mu>0.2</mu>
+                <mu2>1.</mu2>
+                <surface>
+                    <friction>
+                        <ode>
+                        <mu>0.2</mu>
+                        <mu2>1.</mu2>
+                        </ode>
+                    </friction>
+                </surface>
+            </gazebo>
+        </link>
+    </xacro:macro>
+    <xacro:macro name="frictionless_wheel" params="link_name xyz rpy">
+        <link name="${link_name}">
+            <visual>
+                <geometry>
+                    <cylinder radius="${wheel_diameter/2}" length="0.0375"/>
+                </geometry>
+                <material name="blue"/>
+                <origin xyz="${xyz}" rpy="${rpy}"/>
+            </visual>
+            <collision>
+                <geometry>
+                    <cylinder radius="${wheel_diameter/2}" length="0.0375"/>
+                </geometry>
+                <origin xyz="${xyz}" rpy="${rpy}"/>
+            </collision>
+            <xacro:cylinder_inertia m="0.1" r="${wheel_diameter/2}" l="0.0375" xyz="${xyz}" rpy="${rpy}"/>
+            <gazebo>
+                <material>Gazebo/Blue</material>
+                <mu>0.2</mu>
+                <mu2>1.</mu2>
+                <surface>
+                    <friction>
+                        <ode>
+                        <mu>0.2</mu>
+                        <mu2>1.</mu2>
+                        </ode>
+                    </friction>
+                </surface>
+            </gazebo>
+        </link>
+    </xacro:macro>
+    <!-- <xacro:macro name="omni_wheel" params="link_name xyz rpy">
+        <link name="${link_name}">
+            <visual>
+                <geometry>
+                    <cylinder radius="${wheel_diameter/2}" length="0.0375"/>
+                </geometry>
+                <material name="gray"/>
+                <origin xyz="${xyz}" rpy="${rpy}"/>
+            </visual>
+            <collision>
+                <geometry>
+                    <cylinder radius="${wheel_diameter/2}" length="0.0375"/>
+                </geometry>
+                <origin xyz="${xyz}" rpy="${rpy}"/>
+            </collision>
+            <xacro:cylinder_inertia m="0.1" r="${wheel_diameter/2}" l="0.0375" xyz="${xyz}" rpy="${rpy}"/>
+        </link>
+    </xacro:macro> -->
 </robot>

File: dev_ws/src/alpay_description/urdf/mobile_base_gazebo.xacro (robot description, xacro)
@@ -2,142 +2,51 @@
 <robot xmlns:xacro="http://www.ros.org/wiki/xacro">
   <link name="base_footprint" />
-  <xacro:property name="base_z" value="0.2" />
-  <link name="base_link">
-    <visual>
-      <geometry>
-        <box size="0.72 0.54  ${base_z}" />
-      </geometry>
-      <material name="white" />
-      <origin xyz="0 0 ${base_z/2}" rpy="0 0 0" />
-    </visual>
-    <collision>
-      <geometry>
-        <box size="0.72 0.54  ${base_z}" />
-      </geometry>
-      <origin xyz="0 0 ${base_z/2}" rpy="0 0 0" />
-    </collision>
-    <xacro:box_inertia m="0.5" x="0.72" y="0.54" z="${base_z}" xyz="0 0 ${base_z/2}" rpy="0 0 0" />
-  </link>
+  <xacro:property name="wheel_diameter" value="0.1"/>
+  <xacro:property name="wheel_length" value="0.044"/>
+  <xacro:property name="structure_width" value="0.05"/>
+  <xacro:property name="structure_step_width" value="0.025"/>
+  <xacro:structure link_name="base_structure" step="12" xyz="0 0 0" rpy="3.14 0 1.57"/>
   <joint name="base_footprint_joint" type="fixed">
-    <parent link="base_footprint" />
-    <child link="base_link" />
-    <origin xyz="-0.14 0 0.125" rpy="0 0 0" />
+    <parent link="base_footprint"/>
+    <child link="base_structure"/>
+    <origin xyz="0 0 ${wheel_diameter/2}" rpy="0 0 0"/>
   </joint>
-  <link name="base_front">
-    <visual>
-      <geometry>
-        <cylinder radius="0.28" length="${base_z}" />
-      </geometry>
-      <material name="white" />
-      <origin xyz="0 0 ${base_z/2}" rpy="0 0 0" />
-    </visual>
-    <collision>
-      <geometry>
-        <cylinder radius="0.28" length="${base_z}" />
-      </geometry>
-      <origin xyz="0 0 ${base_z/2}" rpy="0 0 0" />
-    </collision>
-    <xacro:cylinder_inertia m="0.2" r="0.28" l="${base_z}" xyz="0 0 ${base_z/2}" rpy="0 0 0" />
-  </link>
-  <joint name="base_front_joint" type="fixed">
-    <parent link="base_link" />
-    <child link="base_front" />
-    <origin xyz="0.28 0 0" rpy="0 0 0" />
+  <xacro:structure link_name="left_structure" step="16" xyz="0 0 0" rpy="3.14 0 0"/>
+  <joint name="left_structure_joint" type="fixed">
+    <parent link="base_structure"/>
+    <child link="left_structure"/>
+    <origin xyz="0 ${structure_step_width*6+structure_width/2} 0" rpy="0 0 0"/>
   </joint>
-  <link name="left_wheel">
-    <visual>
-      <geometry>
-        <cylinder radius="0.125" length="0.05" />
-      </geometry>
-      <material name="black" />
-      <origin xyz="0 0 0" rpy="0 0 0" />
-    </visual>
-    <collision>
-      <geometry>
-        <sphere radius="0.125"/>
-      </geometry>
-      <origin xyz="0 0 0" rpy="0 0 0" />
-    </collision>
-    <xacro:cylinder_inertia m="0.5" r="0.125" l="0.05" xyz="0 0 0" rpy="0 0 0" />
-  </link>
-  <joint name="left_wheel_joint" type="continuous">
-    <parent link="base_link" />
-    <child link="left_wheel" />
-    <origin xyz="0 0.25 0" rpy="1.57 0 3.14" />
+  <xacro:structure link_name="right_structure" step="16" xyz="0 0 0" rpy="3.14 0 0"/>
+  <joint name="right_structure_joint" type="fixed">
+    <parent link="base_structure"/>
+    <child link="right_structure"/>
+    <origin xyz="0 -${structure_step_width*6+structure_width/2} 0" rpy="0 0 0"/>
+  </joint>
+  <xacro:traction_wheel link_name="front_left_wheel" xyz="0 0 0" rpy="0 0 0"/>
+  <joint name="front_left_wheel_joint" type="continuous">
+    <parent link="left_structure"/>
+    <child link="front_left_wheel"/>
+    <origin xyz="${structure_step_width*6} ${structure_width/2+wheel_length/2} 0" rpy="-1.57 0 0"/>
     <axis xyz="0 0 1" />
   </joint>
-  <link name="right_wheel">
-    <visual>
-      <geometry>
-        <cylinder radius="0.125" length="0.05" />
-      </geometry>
-      <material name="black" />
-      <origin xyz="0 0 0" rpy="0 0 0" />
-    </visual>
-    <collision>
-      <geometry>
-        <sphere radius="0.125"/>
-      </geometry>
-      <origin xyz="0 0 0" rpy="0 0 0" />
-    </collision>
-    <xacro:cylinder_inertia m="0.5" r="0.125" l="0.05" xyz="0 0 0" rpy="0 0 0" />
-  </link>
-  <joint name="right_wheel_joint" type="continuous">
-    <parent link="base_link" />
-    <child link="right_wheel" />
-    <origin xyz="0 -0.25 0" rpy="1.57 0 3.14" />
+  <xacro:traction_wheel link_name="front_right_wheel" xyz="0 0 0" rpy="0 0 0"/>
+  <joint name="front_right_wheel_joint" type="continuous">
+    <parent link="right_structure"/>
+    <child link="front_right_wheel"/>
+    <origin xyz="${structure_step_width*6} -${structure_width/2+wheel_length/2} 0" rpy="-1.57 0 0"/>
     <axis xyz="0 0 1" />
   </joint>
-  <link name="brush">
-    <visual>
-      <geometry>
-        <cylinder radius="0.28" length="0.12" />
-      </geometry>
-      <material name="blue" />
-      <origin xyz="0 0 0.06" rpy="0 0 0" />
-    </visual>
-    <collision>
-      <geometry>
-        <sphere radius="0.06"/>
-      </geometry>
-      <origin xyz="0 0 0.06" rpy="0 0 0" />
-    </collision>
-    <xacro:cylinder_inertia m="0.03" r="0.28" l="0.12" xyz="0 0 0.06" rpy="0 0 0" />
-  </link>
-  <joint name="brush_joint" type="fixed">
-    <parent link="base_front" />
-    <child link="brush" />
-    <origin xyz="0.095 0 -0.125" rpy="0 0 0" />
-    <!-- <axis xyz="0 0 1"/> -->
+  <xacro:frictionless_wheel link_name="rear_left_wheel" xyz="0 0 0" rpy="0 0 0"/>
+  <joint name="rear_left_wheel_joint" type="fixed">
+    <parent link="left_structure"/>
+    <child link="rear_left_wheel"/>
+    <origin xyz="-${structure_step_width*6} ${structure_width/2+wheel_length/2} 0" rpy="-1.57 0 0"/>
   </joint>
-  <link name="imu_link" />
-  <joint name="imu_joint" type="fixed">
-    <parent link="base_link" />  <!-- Attach to the appropriate link -->
-    <child link="imu_link" />
-    <origin xyz="0 0 0" rpy="0 0 0" />  <!-- Adjust position -->
-  </joint>
-  <xacro:property name="scan_l" value="0.04" />
-  <xacro:property name="scan_r" value="0.06" />
-  <link name="base_scan">
-    <visual>
-      <geometry>
-        <cylinder radius="${scan_r}" length="${scan_l}" />
-      </geometry>
-      <material name="black" />
-      <origin xyz="0 0 0" rpy="0 0 0" />
-    </visual>
-    <collision>
-      <geometry>
-        <cylinder radius="${scan_r}" length="${scan_l}" />
-      </geometry>
-      <origin xyz="0 0 0" rpy="0 0 0" />
-    </collision>
-    <xacro:cylinder_inertia m="0.04" r="${scan_r}" l="${scan_l}" xyz="0 0 0" rpy="0 0 0" />
-  </link>
-  <joint name="scan_joint" type="fixed">
-    <parent link="base_front" />
-    <child link="base_scan" />
-    <origin xyz="0.15 0 ${base_z+scan_l/2}" rpy="0 0 0" />
-    <!-- <axis xyz="0 0 1"/> -->
+  <xacro:frictionless_wheel link_name="rear_right_wheel" xyz="0 0 0" rpy="0 0 0"/>
+  <joint name="rear_right_wheel_joint" type="fixed">
+    <parent link="right_structure"/>
+    <child link="rear_right_wheel"/>
+    <origin xyz="-${structure_step_width*6} -${structure_width/2+wheel_length/2} 0" rpy="-1.57 0 0"/>
   </joint>
 </robot>

File: dev_ws/src/alpay_description/urdf/ros2_control_gazebo.xacro (robot description, xacro)
@@ -21,8 +21,20 @@
       <state_interface name="position"/>
     </joint>
+    <joint name="left_omni_joint">
+      <state_interface name="velocity"/>
+      <state_interface name="position"/>
+    </joint>
+    <joint name="right_omni_joint">
+      <state_interface name="velocity"/>
+      <state_interface name="position"/>
+    </joint>
+    <joint name="rear_omni_joint">
+      <state_interface name="velocity"/>
+      <state_interface name="position"/>
+    </joint>
   </ros2_control>
   <gazebo>
     <plugin name="gazebo_ros2_control" filename="libgazebo_ros2_control.so">
-      <parameters>$(find cleaner_description)/param/gultepe_controllers1_gazebo.yaml</parameters>
+      <parameters>$(find alpay_description)/param/alpay_controllers_gazebo.yaml</parameters>
     </plugin>
   </gazebo>
