Commit message: Create nfr urdf library

File: dev_ws/src/alpay_description/urdf/alpay_gazebo.urdf.xacro (robot description, xacro)
@@ -2,5 +2,5 @@
 <robot name="alpay" xmlns:xacro="http://www.ros.org/wiki/xacro">
     <xacro:include filename="common.xacro"/>
-    <xacro:include filename="common_gazebo.xacro"/>
+    <xacro:include filename="nfr/nfr_all.xacro"/>
     <xacro:include filename="mobile_base_gazebo.xacro"/>
     <xacro:include filename="sensor_gazebo.xacro"/>

File: dev_ws/src/alpay_description/urdf/common.xacro (robot description, xacro)
@@ -3,5 +3,5 @@
     <material name="red"> <color rgba="0.6 0 0 1"/> </material>
     <material name="green"> <color rgba="0 0.6 0 1"/> </material>
-    <material name="blue"> <color rgba="0 0 0.6 1"/> </material>
+    <material name="blue"> <color rgba="0 0 0.9 1"/> </material>
     <material name="gray"> <color rgba="0.6 0.6 0.6 1"/> </material>
     <material name="light_gray"> <color rgba="0.8 0.8 0.8 1"/> </material>
@@ -35,8 +35,12 @@
             <origin xyz="${xyz}" rpy="${rpy}"/>
             <mass value="${m}"/>
-            <inertia ixx="${m/12*(2*(y*t**3)+(y*(z-2*t)**3))}"
+            <!-- <inertia ixx="${m/12*(2*(y*t**3)+(y*(z-2*t)**3))}"
                      iyy="${m/12*(2*(z*t**3)+(x*(z-2*t)**3))}"
                      izz="${m/12*((x*y**3)-((x-2*t)*(y-2*t)**3))}"
-                     ixy="0" ixz="0" iyz="0"/>
+                     ixy="0" ixz="0" iyz="0"/> -->
+            <inertia ixx="${m*((y*y+z*z)/12-((y-t)*(y-t)*z*z)/(12*(1-(t*y*z)/(x*y*z))))}"
+                iyy="${m*((x*x+z*z)/12-(x*x*(z-t)*(z-t))/(12*(1-(t*x*z)/(x*y*z))))}"
+                izz="${m*((x*x+y*y)/12-(x*x*(y-t)*(y-t))/(12*(1-(t*x*y)/(x*y*z))))}"
+                ixy="0" iyz="0" ixz="0"/>
         </inertial>
     </xacro:macro>
@@ -126,11 +130,11 @@
             <gazebo>
                 <material>Gazebo/Blue</material>
-                <mu>0.2</mu>
-                <mu2>1.</mu2>
+                <mu>0.</mu>
+                <mu2>0.</mu2>
                 <surface>
                     <friction>
                         <ode>
-                        <mu>0.2</mu>
-                        <mu2>1.</mu2>
+                            <mu>0.</mu>
+                            <mu2>0.</mu2>
                         </ode>
                     </friction>
@@ -139,21 +143,3 @@
         </link>
     </xacro:macro>
-    <!-- <xacro:macro name="omni_wheel" params="link_name xyz rpy">
-        <link name="${link_name}">
-            <visual>
-                <geometry>
-                    <cylinder radius="${wheel_diameter/2}" length="0.0375"/>
-                </geometry>
-                <material name="gray"/>
-                <origin xyz="${xyz}" rpy="${rpy}"/>
-            </visual>
-            <collision>
-                <geometry>
-                    <cylinder radius="${wheel_diameter/2}" length="0.0375"/>
-                </geometry>
-                <origin xyz="${xyz}" rpy="${rpy}"/>
-            </collision>
-            <xacro:cylinder_inertia m="0.1" r="${wheel_diameter/2}" l="0.0375" xyz="${xyz}" rpy="${rpy}"/>
-        </link>
-    </xacro:macro> -->
 </robot>

File: dev_ws/src/alpay_description/urdf/mobile_base_gazebo.xacro (robot description, xacro)
@@ -6,5 +6,5 @@
   <xacro:property name="structure_width" value="0.05"/>
   <xacro:property name="structure_step_width" value="0.025"/>
-  <xacro:structure link_name="base_structure" step="12" xyz="0 0 0" rpy="3.14 0 1.57"/>
+  <xacro:nfr_structure link_name="base_structure" step="12" xyz="0 0 0" rpy="3.14 0 1.57"/>
   <joint name="base_footprint_joint" type="fixed">
     <parent link="base_footprint"/>
@@ -12,5 +12,5 @@
     <origin xyz="0 0 ${wheel_diameter/2}" rpy="0 0 0"/>
   </joint>
-  <xacro:structure link_name="left_structure" step="16" xyz="0 0 0" rpy="3.14 0 0"/>
+  <xacro:nfr_structure link_name="left_structure" step="16" xyz="0 0 0" rpy="3.14 0 0"/>
   <joint name="left_structure_joint" type="fixed">
     <parent link="base_structure"/>
@@ -18,5 +18,5 @@
     <origin xyz="0 ${structure_step_width*6+structure_width/2} 0" rpy="0 0 0"/>
   </joint>
-  <xacro:structure link_name="right_structure" step="16" xyz="0 0 0" rpy="3.14 0 0"/>
+  <xacro:nfr_structure link_name="right_structure" step="16" xyz="0 0 0" rpy="3.14 0 0"/>
   <joint name="right_structure_joint" type="fixed">
     <parent link="base_structure"/>
@@ -29,5 +29,5 @@
     <child link="front_left_wheel"/>
     <origin xyz="${structure_step_width*6} ${structure_width/2+wheel_length/2} 0" rpy="-1.57 0 0"/>
-    <axis xyz="0 0 1" />
+    <axis xyz="0 0 1"/>
   </joint>
   <xacro:traction_wheel link_name="front_right_wheel" xyz="0 0 0" rpy="0 0 0"/>
@@ -36,5 +36,5 @@
     <child link="front_right_wheel"/>
     <origin xyz="${structure_step_width*6} -${structure_width/2+wheel_length/2} 0" rpy="-1.57 0 0"/>
-    <axis xyz="0 0 1" />
+    <axis xyz="0 0 1"/>
   </joint>
   <xacro:frictionless_wheel link_name="rear_left_wheel" xyz="0 0 0" rpy="0 0 0"/>
@@ -50,3 +50,9 @@
     <origin xyz="-${structure_step_width*6} -${structure_width/2+wheel_length/2} 0" rpy="-1.57 0 0"/>
   </joint>
+  <xacro:nfr_mecanum_wheel_l link_name="mecanum_test" xyz="0 0 0" rpy="0 0 0"/>
+  <joint name="mecanum_test_joint" type="fixed">
+    <parent link="base_structure"/>
+    <child link="mecanum_test"/>
+    <origin xyz="0 0 0.3" rpy="0 0 0"/>
+  </joint>
 </robot>
