Commit message: Fix new nfr library

File: dev_ws/src/alpay_description/urdf/mobile_base_gazebo.xacro (robot description, xacro)
@@ -50,8 +50,8 @@
     <origin xyz="-${structure_step_width*6} -${structure_width/2+wheel_length/2} 0" rpy="-1.57 0 0"/>
   </joint>
-  <xacro:nfr_mecanum_wheel_l link_name="mecanum_test" xyz="0 0 0" rpy="0 0 0"/>
+  <xacro:nfr_omni_wheel link_name="omni_test" xyz="0 0 0" rpy="0 0 0"/>
   <joint name="mecanum_test_joint" type="fixed">
     <parent link="base_structure"/>
-    <child link="mecanum_test"/>
+    <child link="omni_test"/>
     <origin xyz="0 0 0.3" rpy="0 0 0"/>
   </joint>

File: dev_ws/src/alpay_description/urdf/nfr/nfr_all.xacro (robot description, xacro)
@@ -3,5 +3,7 @@
     <xacro:include filename="nfr_common.xacro"/>
     <xacro:include filename="nfr_frictionless_wheel.xacro"/>
-    <xacro:include filename="nfr_mecanum_wheel.xacro"/>
+    <xacro:include filename="nfr_mecanum_wheel_l.xacro"/>
+    <xacro:include filename="nfr_mecanum_wheel_r.xacro"/>
+    <xacro:include filename="nfr_omni_wheel.xacro"/>
     <xacro:include filename="nfr_structure.xacro"/>
     <xacro:include filename="nfr_traction_wheel.xacro"/>

File: dev_ws/src/alpay_description/urdf/nfr/nfr_omni_wheel.xacro (robot description, xacro)
@@ -50,5 +50,5 @@
             <parent link="${link_name}"/>
             <child link="${link_name}_roller0"/>
-            <origin xyz="0.043 0 0" rpy="0.85 0 0"/>
+            <origin xyz="0.043 0 0" rpy="1.57 0 0"/>
             <axis xyz="0 0 1"/>
         </joint>
