Commit message: Remove origin parameters from omni

File: dev_ws/src/diffbot_description/urdf/nfr/nfr_omni_wheel.xacro (robot description, xacro)
@@ -5,6 +5,6 @@
     <xacro:property name="nfr_roller_radius" value="0.007"/>
     <xacro:property name="nfr_roller_sep_z" value="0.002"/>
-    <xacro:property name="nfr_roller_len" value="0.03"/>
-    <xacro:macro name="nfr_omni_wheel" params="link_name xyz rpy">
+    <xacro:property name="nfr_roller_len" value="0.026"/>
+    <xacro:macro name="nfr_omni_wheel" params="link_name">
         <link name="${link_name}">
             <visual>
@@ -13,7 +13,7 @@
                 </geometry>
                 <material name="nfr_black"/>
-                <origin xyz="${xyz}" rpy="${rpy}"/>
-            </visual>
-            <!-- not necessary, we are sorrounded by rollers anyway -->
+                <origin xyz="0 0 0" rpy="0 0 0"/>
+            </visual>
+            <!-- not necessary since we are sorrounded by rollers anyway -->
             <!-- <collision>
                 <geometry>
@@ -22,5 +22,5 @@
                 <origin xyz="${xyz}" rpy="${rpy}"/>
             </collision> -->
-            <xacro:nfr_cylinder_inertia m="0.180" r="0.042" l="0.0375" xyz="${xyz}" rpy="${rpy}"/>
+            <xacro:nfr_cylinder_inertia m="0.180" r="0.042" l="0.0375" xyz="0 0 0" rpy="0 0 0"/>
         </link>
         <gazebo reference="${link_name}">
@@ -33,15 +33,15 @@
                 </geometry>
                 <material name="nfr_blue"/>
-                <origin xyz="${xyz}" rpy="${rpy}"/>
-            </visual>
-            <collision>
-                <geometry>
-                    <cylinder radius="${nfr_roller_radius}" length="${nfr_roller_len}"/>
-                </geometry>
-                <origin xyz="${xyz}" rpy="${rpy}"/>
-            </collision>
-            <xacro:nfr_cylinder_inertia m="0.006" r="${nfr_roller_radius}" l="${nfr_roller_len}" xyz="${xyz}" rpy="${rpy}"/>
-        </link>
-        <gazebo name="${link_name}_roller0">
+                <origin xyz="0 0 0" rpy="0 0 0"/>
+            </visual>
+            <collision>
+                <geometry>
+                    <cylinder radius="${nfr_roller_radius}" length="${nfr_roller_len}"/>
+                </geometry>
+                <origin xyz="0 0 0" rpy="0 0 0"/>
+            </collision>
+            <xacro:nfr_cylinder_inertia m="0.006" r="${nfr_roller_radius}" l="${nfr_roller_len}" xyz="0 0 0" rpy="0 0 0"/>
+        </link>
+        <gazebo reference="${link_name}_roller0">
             <material>Gazebo/Blue</material>
             <mu>${nfr_roller_friction_mu}</mu>
@@ -68,13 +68,13 @@
                 </geometry>
                 <material name="nfr_blue"/>
-                <origin xyz="${xyz}" rpy="${rpy}"/>
-            </visual>
-            <collision>
-                <geometry>
-                    <cylinder radius="${nfr_roller_radius}" length="${nfr_roller_len}"/>
-                </geometry>
-                <origin xyz="${xyz}" rpy="${rpy}"/>
-            </collision>
-            <xacro:nfr_cylinder_inertia m="0.006" r="${nfr_roller_radius}" l="${nfr_roller_len}" xyz="${xyz}" rpy="${rpy}"/>
+                <origin xyz="0 0 0" rpy="0 0 0"/>
+            </visual>
+            <collision>
+                <geometry>
+                    <cylinder radius="${nfr_roller_radius}" length="${nfr_roller_len}"/>
+                </geometry>
+                <origin xyz="0 0 0" rpy="0 0 0"/>
+            </collision>
+            <xacro:nfr_cylinder_inertia m="0.006" r="${nfr_roller_radius}" l="${nfr_roller_len}" xyz="0 0 0" rpy="0 0 0"/>
         </link>
         <gazebo reference="${link_name}_roller1">
@@ -103,13 +103,13 @@
                 </geometry>
                 <material name="nfr_blue"/>
-                <origin xyz="${xyz}" rpy="${rpy}"/>
-            </visual>
-            <collision>
-                <geometry>
-                    <cylinder radius="${nfr_roller_radius}" length="${nfr_roller_len}"/>
-                </geometry>
-                <origin xyz="${xyz}" rpy="${rpy}"/>
-            </collision>
-            <xacro:nfr_cylinder_inertia m="0.006" r="${nfr_roller_radius}" l="${nfr_roller_len}" xyz="${xyz}" rpy="${rpy}"/>
+                <origin xyz="0 0 0" rpy="0 0 0"/>
+            </visual>
+            <collision>
+                <geometry>
+                    <cylinder radius="${nfr_roller_radius}" length="${nfr_roller_len}"/>
+                </geometry>
+                <origin xyz="0 0 0" rpy="0 0 0"/>
+            </collision>
+            <xacro:nfr_cylinder_inertia m="0.006" r="${nfr_roller_radius}" l="${nfr_roller_len}" xyz="0 0 0" rpy="0 0 0"/>
         </link>
         <gazebo reference="${link_name}_roller2">
@@ -138,13 +138,13 @@
                 </geometry>
                 <material name="nfr_blue"/>
-                <origin xyz="${xyz}" rpy="${rpy}"/>
-            </visual>
-            <collision>
-                <geometry>
-                    <cylinder radius="${nfr_roller_radius}" length="${nfr_roller_len}"/>
-                </geometry>
-                <origin xyz="${xyz}" rpy="${rpy}"/>
-            </collision>
-            <xacro:nfr_cylinder_inertia m="0.006" r="${nfr_roller_radius}" l="${nfr_roller_len}" xyz="${xyz}" rpy="${rpy}"/>
+                <origin xyz="0 0 0" rpy="0 0 0"/>
+            </visual>
+            <collision>
+                <geometry>
+                    <cylinder radius="${nfr_roller_radius}" length="${nfr_roller_len}"/>
+                </geometry>
+                <origin xyz="0 0 0" rpy="0 0 0"/>
+            </collision>
+            <xacro:nfr_cylinder_inertia m="0.006" r="${nfr_roller_radius}" l="${nfr_roller_len}" xyz="0 0 0" rpy="0 0 0"/>
         </link>
         <gazebo reference="${link_name}_roller3">
@@ -173,13 +173,13 @@
                 </geometry>
                 <material name="nfr_blue"/>
-                <origin xyz="${xyz}" rpy="${rpy}"/>
-            </visual>
-            <collision>
-                <geometry>
-                    <cylinder radius="${nfr_roller_radius}" length="${nfr_roller_len}"/>
-                </geometry>
-                <origin xyz="${xyz}" rpy="${rpy}"/>
-            </collision>
-            <xacro:nfr_cylinder_inertia m="0.006" r="${nfr_roller_radius}" l="${nfr_roller_len}" xyz="${xyz}" rpy="${rpy}"/>
+                <origin xyz="0 0 0" rpy="0 0 0"/>
+            </visual>
+            <collision>
+                <geometry>
+                    <cylinder radius="${nfr_roller_radius}" length="${nfr_roller_len}"/>
+                </geometry>
+                <origin xyz="0 0 0" rpy="0 0 0"/>
+            </collision>
+            <xacro:nfr_cylinder_inertia m="0.006" r="${nfr_roller_radius}" l="${nfr_roller_len}" xyz="0 0 0" rpy="0 0 0"/>
         </link>
         <gazebo reference="${link_name}_roller4">
@@ -208,13 +208,13 @@
                 </geometry>
                 <material name="nfr_blue"/>
-                <origin xyz="${xyz}" rpy="${rpy}"/>
-            </visual>
-            <collision>
-                <geometry>
-                    <cylinder radius="${nfr_roller_radius}" length="${nfr_roller_len}"/>
-                </geometry>
-                <origin xyz="${xyz}" rpy="${rpy}"/>
-            </collision>
-            <xacro:nfr_cylinder_inertia m="0.006" r="${nfr_roller_radius}" l="${nfr_roller_len}" xyz="${xyz}" rpy="${rpy}"/>
+                <origin xyz="0 0 0" rpy="0 0 0"/>
+            </visual>
+            <collision>
+                <geometry>
+                    <cylinder radius="${nfr_roller_radius}" length="${nfr_roller_len}"/>
+                </geometry>
+                <origin xyz="0 0 0" rpy="0 0 0"/>
+            </collision>
+            <xacro:nfr_cylinder_inertia m="0.006" r="${nfr_roller_radius}" l="${nfr_roller_len}" xyz="0 0 0" rpy="0 0 0"/>
         </link>
         <gazebo reference="${link_name}_roller5">
@@ -243,13 +243,13 @@
                 </geometry>
                 <material name="nfr_blue"/>
-                <origin xyz="${xyz}" rpy="${rpy}"/>
-            </visual>
-            <collision>
-                <geometry>
-                    <cylinder radius="${nfr_roller_radius}" length="${nfr_roller_len}"/>
-                </geometry>
-                <origin xyz="${xyz}" rpy="${rpy}"/>
-            </collision>
-            <xacro:nfr_cylinder_inertia m="0.006" r="${nfr_roller_radius}" l="${nfr_roller_len}" xyz="${xyz}" rpy="${rpy}"/>
+                <origin xyz="0 0 0" rpy="0 0 0"/>
+            </visual>
+            <collision>
+                <geometry>
+                    <cylinder radius="${nfr_roller_radius}" length="${nfr_roller_len}"/>
+                </geometry>
+                <origin xyz="0 0 0" rpy="0 0 0"/>
+            </collision>
+            <xacro:nfr_cylinder_inertia m="0.006" r="${nfr_roller_radius}" l="${nfr_roller_len}" xyz="0 0 0" rpy="0 0 0"/>
         </link>
         <gazebo reference="${link_name}_roller6">
@@ -278,13 +278,13 @@
                 </geometry>
                 <material name="nfr_blue"/>
-                <origin xyz="${xyz}" rpy="${rpy}"/>
-            </visual>
-            <collision>
-                <geometry>
-                    <cylinder radius="${nfr_roller_radius}" length="${nfr_roller_len}"/>
-                </geometry>
-                <origin xyz="${xyz}" rpy="${rpy}"/>
-            </collision>
-            <xacro:nfr_cylinder_inertia m="0.006" r="${nfr_roller_radius}" l="${nfr_roller_len}" xyz="${xyz}" rpy="${rpy}"/>
+                <origin xyz="0 0 0" rpy="0 0 0"/>
+            </visual>
+            <collision>
+                <geometry>
+                    <cylinder radius="${nfr_roller_radius}" length="${nfr_roller_len}"/>
+                </geometry>
+                <origin xyz="0 0 0" rpy="0 0 0"/>
+            </collision>
+            <xacro:nfr_cylinder_inertia m="0.006" r="${nfr_roller_radius}" l="${nfr_roller_len}" xyz="0 0 0" rpy="0 0 0"/>
         </link>
         <gazebo reference="${link_name}_roller7">
@@ -313,13 +313,13 @@
                 </geometry>
                 <material name="nfr_blue"/>
-                <origin xyz="${xyz}" rpy="${rpy}"/>
-            </visual>
-            <collision>
-                <geometry>
-                    <cylinder radius="${nfr_roller_radius}" length="${nfr_roller_len}"/>
-                </geometry>
-                <origin xyz="${xyz}" rpy="${rpy}"/>
-            </collision>
-            <xacro:nfr_cylinder_inertia m="0.006" r="${nfr_roller_radius}" l="${nfr_roller_len}" xyz="${xyz}" rpy="${rpy}"/>
+                <origin xyz="0 0 0" rpy="0 0 0"/>
+            </visual>
+            <collision>
+                <geometry>
+                    <cylinder radius="${nfr_roller_radius}" length="${nfr_roller_len}"/>
+                </geometry>
+                <origin xyz="0 0 0" rpy="0 0 0"/>
+            </collision>
+            <xacro:nfr_cylinder_inertia m="0.006" r="${nfr_roller_radius}" l="${nfr_roller_len}" xyz="0 0 0" rpy="0 0 0"/>
         </link>
         <gazebo reference="${link_name}_roller8">
@@ -348,13 +348,13 @@
                 </geometry>
                 <material name="nfr_blue"/>
-                <origin xyz="${xyz}" rpy="${rpy}"/>
-            </visual>
-            <collision>
-                <geometry>
-                    <cylinder radius="${nfr_roller_radius}" length="${nfr_roller_len}"/>
-                </geometry>
-                <origin xyz="${xyz}" rpy="${rpy}"/>
-            </collision>
-            <xacro:nfr_cylinder_inertia m="0.006" r="${nfr_roller_radius}" l="${nfr_roller_len}" xyz="${xyz}" rpy="${rpy}"/>
+                <origin xyz="0 0 0" rpy="0 0 0"/>
+            </visual>
+            <collision>
+                <geometry>
+                    <cylinder radius="${nfr_roller_radius}" length="${nfr_roller_len}"/>
+                </geometry>
+                <origin xyz="0 0 0" rpy="0 0 0"/>
+            </collision>
+            <xacro:nfr_cylinder_inertia m="0.006" r="${nfr_roller_radius}" l="${nfr_roller_len}" xyz="0 0 0" rpy="0 0 0"/>
         </link>
         <gazebo reference="${link_name}_roller9">
@@ -383,13 +383,13 @@
                 </geometry>
                 <material name="nfr_blue"/>
-                <origin xyz="${xyz}" rpy="${rpy}"/>
-            </visual>
-            <collision>
-                <geometry>
-                    <cylinder radius="${nfr_roller_radius}" length="${nfr_roller_len}"/>
-                </geometry>
-                <origin xyz="${xyz}" rpy="${rpy}"/>
-            </collision>
-            <xacro:nfr_cylinder_inertia m="0.006" r="${nfr_roller_radius}" l="${nfr_roller_len}" xyz="${xyz}" rpy="${rpy}"/>
+                <origin xyz="0 0 0" rpy="0 0 0"/>
+            </visual>
+            <collision>
+                <geometry>
+                    <cylinder radius="${nfr_roller_radius}" length="${nfr_roller_len}"/>
+                </geometry>
+                <origin xyz="0 0 0" rpy="0 0 0"/>
+            </collision>
+            <xacro:nfr_cylinder_inertia m="0.006" r="${nfr_roller_radius}" l="${nfr_roller_len}" xyz="0 0 0" rpy="0 0 0"/>
         </link>
         <gazebo reference="${link_name}_roller10">
@@ -418,13 +418,13 @@
                 </geometry>
                 <material name="nfr_blue"/>
-                <origin xyz="${xyz}" rpy="${rpy}"/>
-            </visual>
-            <collision>
-                <geometry>
-                    <cylinder radius="${nfr_roller_radius}" length="${nfr_roller_len}"/>
-                </geometry>
-                <origin xyz="${xyz}" rpy="${rpy}"/>
-            </collision>
-            <xacro:nfr_cylinder_inertia m="0.006" r="${nfr_roller_radius}" l="${nfr_roller_len}" xyz="${xyz}" rpy="${rpy}"/>
+                <origin xyz="0 0 0" rpy="0 0 0"/>
+            </visual>
+            <collision>
+                <geometry>
+                    <cylinder radius="${nfr_roller_radius}" length="${nfr_roller_len}"/>
+                </geometry>
+                <origin xyz="0 0 0" rpy="0 0 0"/>
+            </collision>
+            <xacro:nfr_cylinder_inertia m="0.006" r="${nfr_roller_radius}" l="${nfr_roller_len}" xyz="0 0 0" rpy="0 0 0"/>
         </link>
         <gazebo reference="${link_name}_roller11">
