Commit message: Update and move struct inertia function

File: dev_ws/src/diffbot_description/urdf/nfr/nfr_common.xacro (robot description, xacro)
@@ -25,11 +25,4 @@
         </inertial>
     </xacro:macro>
-    <xacro:macro name="nfr_struct_inertia" params="step xyz rpy">
-        <!-- structureın uzun kısmı için x ekseni kullanılıyor -->
-        <!-- boş olan taraf üste (+z) bakıyor -->
-        <!-- şimdilik böyle yapıyorum affedin beni -->
-        <xacro:nfr_box_inertia m="${step*0.016}" x="${step*0.025}"
-                                   y="0.05" z="0.05" xyz="${xyz}" rpy="${rpy}"/>
-    </xacro:macro>
     <xacro:macro name="nfr_cylinder_inertia" params="m r l xyz rpy">
         <inertial>

File: dev_ws/src/diffbot_description/urdf/nfr/nfr_structure.xacro (robot description, xacro)
@@ -5,5 +5,5 @@
         <!-- boş olan taraf üste (+z) bakıyor -->
         <!-- şimdilik böyle yapıyorum affedin beni -->
-        <xacro:nfr_box_inertia m="${step*0.016}" x="${step*0.025}"
+        <xacro:nfr_box_inertia m="${step*0.020}" x="${step*0.025}"
                                    y="0.05" z="0.05" xyz="${xyz}" rpy="${rpy}"/>
     </xacro:macro>
