Commit message: Remove parameters and fix frictionless and traction wheels

File: dev_ws/src/diffbot_description/urdf/nfr/nfr_frictionless_wheel.xacro (robot description, xacro)
@@ -2,5 +2,5 @@
 <robot xmlns:xacro="http://www.ros.org/wiki/xacro">
     <xacro:property name="nfr_wheel_diam" value="0.1"/>
-    <xacro:macro name="nfr_frictionless_wheel" params="link_name xyz rpy">
+    <xacro:macro name="nfr_frictionless_wheel" params="link_name">
         <link name="${link_name}">
             <visual>
@@ -9,5 +9,5 @@
                 </geometry>
                 <material name="nfr_blue"/>
-                <origin xyz="${xyz}" rpy="${rpy}"/>
+                <origin xyz="0 0 0" rpy="0 0 0"/>
             </visual>
             <collision>
@@ -15,9 +15,9 @@
                     <cylinder radius="${nfr_wheel_diam/2}" length="0.0375"/>
                 </geometry>
-                <origin xyz="${xyz}" rpy="${rpy}"/>
+                <origin xyz="0 0 0" rpy="0 0 0"/>
             </collision>
-            <xacro:nfr_cylinder_inertia m="0.1" r="${nfr_wheel_diam/2}" l="0.0375" xyz="${xyz}" rpy="${rpy}"/>
+            <xacro:nfr_cylinder_inertia m="0.1" r="${nfr_wheel_diam/2}" l="0.0375" xyz="0 0 0" rpy="0 0 0"/>
         </link>
-        <gazebo reference="nfr_frictionless_wheel">
+        <gazebo reference="${link_name}">
             <material>Gazebo/Blue</material>
             <mu>0.</mu>

File: dev_ws/src/diffbot_description/urdf/nfr/nfr_traction_wheel.xacro (robot description, xacro)
@@ -4,5 +4,5 @@
     <xacro:property name="nfr_trac_fric_mu2" value="1"/>
     <xacro:property name="nfr_wheel_diam" value="0.1"/>
-    <xacro:macro name="nfr_traction_wheel" params="link_name xyz rpy">
+    <xacro:macro name="nfr_traction_wheel" params="link_name">
         <link name="${link_name}">
             <visual>
@@ -11,5 +11,5 @@
                 </geometry>
                 <material name="nfr_gray"/>
-                <origin xyz="${xyz}" rpy="${rpy}"/>
+                <origin xyz="0 0 0" rpy="0 0 0"/>
             </visual>
             <collision>
@@ -17,9 +17,9 @@
                     <cylinder radius="${nfr_wheel_diam/2}" length="0.0375"/>
                 </geometry>
-                <origin xyz="${xyz}" rpy="${rpy}"/>
+                <origin xyz="0 0 0" rpy="0 0 0"/>
             </collision>
-            <xacro:nfr_cylinder_inertia m="0.1" r="${nfr_wheel_diam/2}" l="0.0375" xyz="${xyz}" rpy="${rpy}"/>
+            <xacro:nfr_cylinder_inertia m="0.1" r="${nfr_wheel_diam/2}" l="0.0375" xyz="0 0 0" rpy="0 0 0"/>
         </link>
-        <gazebo reference="nfr_traction_wheel">
+        <gazebo reference="${link_name}">
             <material>Gazebo/Gray</material>
             <mu>${nfr_trac_fric_mu}</mu>
