Commit message: Debug unexpected simulation behaviour

File: dev_ws/src/diffbot_description/urdf/mobile_base_gazebo.xacro (robot description, xacro)
@@ -11,5 +11,5 @@
     <parent link="base_footprint"/>
     <child link="front_structure"/>
-    <origin xyz="${structure_step_width*3} 0 ${wheel_diameter/2}" rpy="0 0 0"/>
+    <origin xyz="${structure_step_width*1} 0 ${wheel_diameter/2}" rpy="0 0 0"/>
   </joint>
   <xacro:nfr_structure link_name="rear_structure" step="12" xyz="0 0 0" rpy="3.14 0 1.57"/>
@@ -23,5 +23,5 @@
     <parent link="front_structure"/>
     <child link="left_structure"/>
-    <origin xyz="-${structure_step_width*3} ${structure_step_width*6+structure_width/2} 0" rpy="0 0 0"/>
+    <origin xyz="-${structure_step_width*1} ${structure_step_width*6+structure_width/2} 0" rpy="0 0 0"/>
   </joint>
   <xacro:nfr_structure link_name="right_structure" step="16" xyz="0 0 0" rpy="3.14 0 0"/>
@@ -29,8 +29,10 @@
     <parent link="front_structure"/>
     <child link="right_structure"/>
-    <origin xyz="-${structure_step_width*3} -${structure_step_width*6+structure_width/2} 0" rpy="0 0 0"/>
+    <origin xyz="-${structure_step_width*1} -${structure_step_width*6+structure_width/2} 0" rpy="0 0 0"/>
   </joint>
   <!-- Caution, hot wheels -->
-  <xacro:nfr_omni_wheel link_name="front_left_wheel"/>
+  <!-- herkese dağıttığımız şase gibi yapacaktım ama omniler daha mükemmel değil o
+  yüzden sürtünmesiz teker kullandım. onda da drop center yapmam gerekiyor -->
+  <!-- <xacro:nfr_frictionless_wheel link_name="front_left_wheel"/>
   <joint name="front_left_wheel_joint" type="continuous">
     <parent link="left_structure"/>
@@ -38,6 +40,6 @@
     <origin xyz="${structure_step_width*6} ${structure_width/2+wheel_length/2} 0" rpy="-1.57 0 0"/>
     <axis xyz="0 0 1"/>
-  </joint>
-  <xacro:nfr_omni_wheel link_name="front_right_wheel"/>
+  </joint> -->
+  <!-- <xacro:nfr_frictionless_wheel  link_name="front_right_wheel"/>
   <joint name="front_right_wheel_joint" type="continuous">
     <parent link="right_structure"/>
@@ -45,11 +47,13 @@
     <origin xyz="${structure_step_width*6} -${structure_width/2+wheel_length/2} 0" rpy="-1.57 0 0"/>
     <axis xyz="0 0 1"/>
-  </joint>
+  </joint> -->
   <xacro:nfr_traction_wheel link_name="left_wheel"/>
   <joint name="left_wheel_joint" type="continuous">
     <parent link="left_structure"/>
     <child link="left_wheel"/>
-    <origin xyz="0 ${structure_width/2+wheel_length/2} 0" rpy="-1.57 0 0"/>
+    <origin xyz="${structure_step_width*6} ${structure_width/2+wheel_length/2} 0" rpy="-1.57 0 0"/>
+    <!-- <origin xyz="0 ${structure_width/2+wheel_length/2} 0" rpy="-1.57 0 0"/> -->
     <axis xyz="0 0 1"/>
+    <limit effort="500.0" velocity="10.0" />
   </joint>
   <xacro:nfr_traction_wheel link_name="right_wheel"/>
@@ -57,18 +61,24 @@
     <parent link="right_structure"/>
     <child link="right_wheel"/>
-    <origin xyz="0 -${structure_width/2+wheel_length/2} 0" rpy="-1.57 0 0"/>
-    <axis xyz="0 0 1"/>
+    <origin xyz="${structure_step_width*6} -${structure_width/2+wheel_length/2} 0" rpy="-4.71 0 0"/>
+    <!-- <origin xyz="0 -${structure_width/2+wheel_length/2} 0" rpy="-1.57 0 0"/> -->
+    <axis xyz="0 0 -1"/>
+    <limit effort="500.0" velocity="10.0" />
   </joint>
-  <xacro:nfr_omni_wheel link_name="rear_left_wheel"/>
-  <joint name="rear_left_wheel_joint" type="fixed">
+  <xacro:nfr_frictionless_wheel link_name="rear_left_wheel"/>
+  <joint name="rear_left_wheel_joint" type="continuous">
     <parent link="left_structure"/>
     <child link="rear_left_wheel"/>
     <origin xyz="-${structure_step_width*6} ${structure_width/2+wheel_length/2} 0" rpy="-1.57 0 0"/>
+    <axis xyz="0 0 1"/>
+    <limit effort="500.0" velocity="10.0" />
   </joint>
-  <xacro:nfr_omni_wheel link_name="rear_right_wheel"/>
-  <joint name="rear_right_wheel_joint" type="fixed">
+  <xacro:nfr_frictionless_wheel link_name="rear_right_wheel"/>
+  <joint name="rear_right_wheel_joint" type="continuous">
     <parent link="right_structure"/>
     <child link="rear_right_wheel"/>
-    <origin xyz="-${structure_step_width*6} -${structure_width/2+wheel_length/2} 0" rpy="-1.57 0 0"/>
+    <origin xyz="-${structure_step_width*6} -${structure_width/2+wheel_length/2} 0" rpy="-4.71 0 0"/>
+    <axis xyz="0 0 -1"/>
+    <limit effort="500.0" velocity="10.0" />
   </joint>
   <!-- electronics -->
@@ -76,5 +86,5 @@
       <visual>
           <geometry>
-              <box size="${structure_step_width*10} ${structure_step_width*12} 0.004"/>
+              <box size="${structure_step_width*8} ${structure_step_width*12} 0.004"/>
           </geometry>
           <material name="white"/>
@@ -87,5 +97,5 @@
           <origin xyz="0 0 0" rpy="0 0 0"/>
       </collision> -->
-      <xacro:box_inertia m="0.2" x="${structure_step_width*10}" y="${structure_step_width*12}" z="0.004" xyz="0 0 0" rpy="0 0 0"/>
+      <xacro:box_inertia m="0.2" x="${structure_step_width*8}" y="${structure_step_width*12}" z="0.004" xyz="0 0 0" rpy="0 0 0"/>
   </link>
   <gazebo reference="electronics_base">
@@ -95,7 +105,7 @@
     <parent link="front_structure"/>
     <child link="electronics_base"/>
-    <origin xyz="-${structure_step_width*5} 0 -${structure_step_width+0.004}" rpy="0 0 0"/>
+    <origin xyz="-${structure_step_width*4} 0 -${structure_step_width+0.004}" rpy="0 0 0"/>
   </joint>
-  <link name="battery">
+  <!-- <link name="battery">
       <visual>
           <geometry>
@@ -105,10 +115,4 @@
           <origin xyz="0 0 0" rpy="0 0 0"/>
       </visual>
-      <!-- <collision>
-          <geometry>
-              <box size="0.1135 0.0905 0.023"/>
-          </geometry>
-          <origin xyz="0 0 0" rpy="0 0 0"/>
-      </collision> -->
       <xacro:box_inertia m="0.567" x="0.1135" y="0.0905" z="0.023" xyz="0 0 0" rpy="0 0 0"/>
   </link>
@@ -119,7 +123,7 @@
     <parent link="electronics_base"/>
     <child link="battery"/>
-    <origin xyz="0 0.08475 ${0.004+0.00115}" rpy="0 0 0"/>
-  </joint>
-  <link name="control_hub">
+    <origin xyz="0 0.08475 ${0.004+0.0115}" rpy="0 0 0"/>
+  </joint> -->
+  <!-- <link name="control_hub">
       <visual>
           <geometry>
@@ -129,10 +133,4 @@
           <origin xyz="0 0 0" rpy="0 0 0"/>
       </visual>
-      <!-- <collision>
-          <geometry>
-              <box size="0.143 0.103 0.0295"/>
-          </geometry>
-          <origin xyz="0 0 0" rpy="0 0 0"/>
-      </collision> -->
       <xacro:box_inertia m="0.209" x="0.143" y="0.103" z="0.0295" xyz="0 0 0" rpy="0 0 0"/>
   </link>
@@ -144,5 +142,47 @@
     <child link="control_hub"/>
     <origin xyz="0 -0.0785 ${0.004+0.01475}" rpy="0 0 0"/>
-  </joint>
+  </joint> -->
   <!-- odom pod omni wheels -->
+  <!-- <xacro:nfr_odometry_pod link_name="left_odom"/>
+  <joint name="left_odom_joint" type="fixed">
+    <parent link="front_structure"/>
+    <child link="left_odom"/>
+    <origin xyz="${structure_step_width} ${structure_step_width*5} 0" rpy="0 0 0"/>
+  </joint> -->
+  <!-- <xacro:nfr_odometry_pod link_name="right_odom"/>
+  <joint name="right_odom_joint" type="fixed">
+    <parent link="front_structure"/>
+    <child link="right_odom"/>
+    <origin xyz="${structure_step_width} -${structure_step_width*5} 0" rpy="0 0 0"/>
+  </joint> -->
+  <!-- <xacro:nfr_structure link_name="rear_odom_base" step="2" xyz="0 0 0" rpy="0 0 0"/>
+  <joint name="rear_odom_base_joint" type="fixed">
+    <parent link="front_structure"/>
+    <child link="rear_odom_base"/>
+    <origin xyz="${structure_step_width*2} ${-0.04-structure_step_width} 0" rpy="0 0 0"/>
+  </joint> -->
+  <!-- <xacro:nfr_odometry_pod link_name="rear_odom"/>
+  <joint name="rear_odom_joint" type="fixed">
+    <parent link="rear_odom_base"/>
+    <child link="rear_odom"/>
+    <origin xyz="0 ${structure_step_width} 0" rpy="0 0 1.57"/>
+  </joint> -->
+  <!-- <link name="weight">
+      <visual>
+          <geometry>
+              <box size="0.05 0.05 0.05"/>
+          </geometry>
+          <material name="black"/>
+          <origin xyz="0 0 0" rpy="0 0 0"/>
+      </visual>
+      <xacro:box_inertia m="3" x="0.05" y="0.05" z="0.05" xyz="0 0 0" rpy="0 0 0"/>
+  </link>
+  <gazebo reference="weight">
+      <material>Gazebo/Black</material>
+  </gazebo>
+  <joint name="weight_joint" type="fixed">
+    <parent link="front_structure"/>
+    <child link="weight"/>
+    <origin xyz="0 0 ${structure_step_width*2}" rpy="0 0 0"/>
+  </joint> -->
 </robot>

File: dev_ws/src/diffbot_description/urdf/nfr/nfr.xacro (robot description, xacro)
@@ -6,4 +6,6 @@
     <xacro:include filename="nfr_mecanum_wheel_r.xacro"/>
     <xacro:include filename="nfr_omni_wheel.xacro"/>
+    <xacro:include filename="nfr_mini_omni_wheel.xacro"/>
+    <xacro:include filename="nfr_odometry_pod.xacro"/>
     <xacro:include filename="nfr_structure.xacro"/>
     <xacro:include filename="nfr_traction_wheel.xacro"/>

File: dev_ws/src/diffbot_description/urdf/nfr/nfr_common.xacro (robot description, xacro)
@@ -4,4 +4,5 @@
     <material name="nfr_black"> <color rgba="0 0 0 1"/> </material>
     <material name="nfr_blue"> <color rgba="0 0 0.9 1"/> </material>
+    <material name="nfr_white"> <color rgba="1 1 1 1"/> </material>
     <xacro:macro name="nfr_box_inertia" params="m x y z xyz rpy">
         <inertial>

File: dev_ws/src/diffbot_description/urdf/nfr/nfr_frictionless_wheel.xacro (robot description, xacro)
@@ -1,4 +1,6 @@
 <?xml version="1.0"?>
 <robot xmlns:xacro="http://www.ros.org/wiki/xacro">
+    <xacro:property name="nfr_fric_fric_mu" value="0.001"/>
+    <xacro:property name="nfr_fric_fric_mu2" value="0.001"/>
     <xacro:property name="nfr_wheel_diam" value="0.1"/>
     <xacro:macro name="nfr_frictionless_wheel" params="link_name">
@@ -13,5 +15,6 @@
             <collision>
                 <geometry>
-                    <cylinder radius="${nfr_wheel_diam/2}" length="0.0375"/>
+                    <!-- <cylinder radius="${nfr_wheel_diam/2}" length="0.0375"/> -->
+                    <sphere radius="${nfr_wheel_diam/2}"/>
                 </geometry>
                 <origin xyz="0 0 0" rpy="0 0 0"/>
@@ -21,11 +24,14 @@
         <gazebo reference="${link_name}">
             <material>Gazebo/Blue</material>
-            <mu>0.</mu>
-            <mu2>0.</mu2>
+            <mu>${nfr_fric_fric_mu}</mu>
+            <mu2>${nfr_fric_fric_mu2}</mu2>
+            <!-- <minDepth>0.001</minDepth> -->
+            <!-- <kp>100000000</kp> -->
+            <!-- <kd>1</kd> -->
             <surface>
                 <friction>
                     <ode>
-                        <mu>0.</mu>
-                        <mu2>0.</mu2>
+                        <mu>${nfr_fric_fric_mu}</mu>
+                        <mu2>${nfr_fric_fric_mu2}</mu2>
                     </ode>
                 </friction>

File: dev_ws/src/diffbot_description/urdf/nfr/nfr_structure.xacro (robot description, xacro)
@@ -5,6 +5,6 @@
         <!-- boş olan taraf üste (+z) bakıyor -->
         <!-- şimdilik böyle yapıyorum affedin beni -->
-        <xacro:nfr_box_inertia m="${step*0.020}" x="${step*0.025}"
-                                   y="0.05" z="0.05" xyz="${xyz}" rpy="${rpy}"/>
+        <!-- <xacro:nfr_box_inertia m="${step*0.020}" x="${step*0.025}" y="0.05" z="0.05" xyz="${xyz}" rpy="${rpy}"/> -->
+        <xacro:nfr_box_inertia m="0.0001" x="${step*0.025}" y="0.05" z="0.05" xyz="${xyz}" rpy="${rpy}"/>
     </xacro:macro>
     <xacro:macro name="nfr_structure" params="link_name step xyz rpy">

File: dev_ws/src/diffbot_description/urdf/nfr/nfr_traction_wheel.xacro (robot description, xacro)
@@ -1,6 +1,6 @@
 <?xml version="1.0"?>
 <robot xmlns:xacro="http://www.ros.org/wiki/xacro">
-    <xacro:property name="nfr_trac_fric_mu" value="1"/>
-    <xacro:property name="nfr_trac_fric_mu2" value="1"/>
+    <xacro:property name="nfr_trac_fric_mu" value="100"/>
+    <xacro:property name="nfr_trac_fric_mu2" value="100"/>
     <xacro:property name="nfr_wheel_diam" value="0.1"/>
     <xacro:macro name="nfr_traction_wheel" params="link_name">
@@ -9,4 +9,5 @@
                 <geometry>
                     <cylinder radius="${nfr_wheel_diam/2}" length="0.0375"/>
+                    <!-- <sphere radius="${nfr_wheel_diam/2}"/> -->
                 </geometry>
                 <material name="nfr_gray"/>
@@ -15,5 +16,6 @@
             <collision>
                 <geometry>
-                    <cylinder radius="${nfr_wheel_diam/2}" length="0.0375"/>
+                    <!-- <cylinder radius="${nfr_wheel_diam/2}" length="0.0375"/> -->
+                    <sphere radius="${nfr_wheel_diam/2}"/>
                 </geometry>
                 <origin xyz="0 0 0" rpy="0 0 0"/>
@@ -25,4 +27,7 @@
             <mu>${nfr_trac_fric_mu}</mu>
             <mu2>${nfr_trac_fric_mu2}</mu2>
+            <minDepth>0.00001</minDepth>
+            <kp>100000000</kp>
+            <kd>1</kd>
             <surface>
                 <friction>
