Commit message: add nfr component library pkg

File: dev_ws/src/diffbot_description/urdf/diffbot.urdf.xacro (robot description, xacro)
@@ -1,6 +1,7 @@
 <?xml version="1.0"?>
 <robot name="diffbot" xmlns:xacro="http://www.ros.org/wiki/xacro">
+    <xacro:property name="nfr_component_lib_path" value="$(find nfr_component_lib)/urdf/nfr.xacro"/>
+    <xacro:include filename="${nfr_component_lib_path}"/>
     <xacro:include filename="common.xacro"/>
-    <xacro:include filename="nfr/nfr.xacro"/>
     <xacro:include filename="mobile_base_gazebo.xacro"/>
     <xacro:include filename="sensor_gazebo.xacro"/>

File: dev_ws/src/diffbot_description/urdf/mobile_base_gazebo.xacro (robot description, xacro)
@@ -34,18 +34,4 @@
   <!-- herkese dağıttığımız şase gibi yapacaktım ama omniler daha mükemmel değil o
   yüzden sürtünmesiz teker kullandım. onda da drop center yapmam gerekiyor -->
-  <!-- <xacro:nfr_frictionless_wheel link_name="front_left_wheel"/>
-  <joint name="front_left_wheel_joint" type="continuous">
-    <parent link="left_structure"/>
-    <child link="front_left_wheel"/>
-    <origin xyz="${structure_step_width*6} ${structure_width/2+wheel_length/2} 0" rpy="-1.57 0 0"/>
-    <axis xyz="0 0 1"/>
-  </joint> -->
-  <!-- <xacro:nfr_frictionless_wheel  link_name="front_right_wheel"/>
-  <joint name="front_right_wheel_joint" type="continuous">
-    <parent link="right_structure"/>
-    <child link="front_right_wheel"/>
-    <origin xyz="${structure_step_width*6} -${structure_width/2+wheel_length/2} 0" rpy="-1.57 0 0"/>
-    <axis xyz="0 0 1"/>
-  </joint> -->
   <xacro:nfr_traction_wheel link_name="left_wheel"/>
   <joint name="left_wheel_joint" type="continuous">
@@ -66,5 +52,5 @@
     <limit effort="500.0" velocity="10.0" />
   </joint>
-  <xacro:nfr_frictionless_wheel link_name="rear_left_wheel"/>
+  <xacro:nfr_omni_test link_name="rear_left_wheel"/>
   <joint name="rear_left_wheel_joint" type="continuous">
     <parent link="left_structure"/>
@@ -74,5 +60,5 @@
     <limit effort="500.0" velocity="10.0" />
   </joint>
-  <xacro:nfr_frictionless_wheel link_name="rear_right_wheel"/>
+  <xacro:nfr_omni_wheel link_name="rear_right_wheel"/>
   <joint name="rear_right_wheel_joint" type="continuous">
     <parent link="right_structure"/>
@@ -148,12 +134,12 @@
     <parent link="front_structure"/>
     <child link="left_odom"/>
-    <origin xyz="${structure_step_width} ${structure_step_width*5} 0" rpy="0 0 0"/>
+    <origin xyz="${structure_step_width} ${structure_step_width*5} 0.01" rpy="0 0 0"/>
   </joint> -->
-  <!-- <xacro:nfr_odometry_pod link_name="right_odom"/>
+  <xacro:nfr_odometry_pod link_name="right_odom"/>
   <joint name="right_odom_joint" type="fixed">
     <parent link="front_structure"/>
     <child link="right_odom"/>
-    <origin xyz="${structure_step_width} -${structure_step_width*5} 0" rpy="0 0 0"/>
-  </joint> -->
+    <origin xyz="${structure_step_width} -${structure_step_width*5} 0.1" rpy="0 0 0"/>
+  </joint>
   <!-- <xacro:nfr_structure link_name="rear_odom_base" step="2" xyz="0 0 0" rpy="0 0 0"/>
   <joint name="rear_odom_base_joint" type="fixed">
@@ -161,12 +147,12 @@
     <child link="rear_odom_base"/>
     <origin xyz="${structure_step_width*2} ${-0.04-structure_step_width} 0" rpy="0 0 0"/>
-  </joint> -->
-  <!-- <xacro:nfr_odometry_pod link_name="rear_odom"/>
+  </joint>
+  <xacro:nfr_odometry_pod link_name="rear_odom"/>
   <joint name="rear_odom_joint" type="fixed">
     <parent link="rear_odom_base"/>
     <child link="rear_odom"/>
-    <origin xyz="0 ${structure_step_width} 0" rpy="0 0 1.57"/>
+    <origin xyz="0 ${structure_step_width} 0.01" rpy="0 0 1.57"/>
   </joint> -->
-  <!-- <link name="weight">
+  <link name="weight">
       <visual>
           <geometry>
@@ -185,4 +171,4 @@
     <child link="weight"/>
     <origin xyz="0 0 ${structure_step_width*2}" rpy="0 0 0"/>
-  </joint> -->
+  </joint>
 </robot>

File: dev_ws/src/nfr_component_lib/urdf/nfr.xacro (robot description, xacro)
@@ -10,3 +10,4 @@
     <xacro:include filename="nfr_structure.xacro"/>
     <xacro:include filename="nfr_traction_wheel.xacro"/>
+    <xacro:include filename="nfr_omni_test.xacro"/>
 </robot>

File: dev_ws/src/nfr_component_lib/urdf/nfr_mini_omni_wheel.xacro (robot description, xacro)
@@ -420,10 +420,10 @@
                 <origin xyz="0 0 0" rpy="0 0 0"/>
             </visual>
-            <collision>
-                <geometry>
-                    <cylinder radius="${nfr_mini_roller_radius}" length="${nfr_mini_roller_len}"/>
-                </geometry>
-                <origin xyz="0 0 0" rpy="0 0 0"/>
-            </collision>
+            <!-- <collision>
+                <geometry>
+                    <cylinder radius="${nfr_mini_roller_radius}" length="${nfr_mini_roller_len}"/>
+                </geometry>
+                <origin xyz="0 0 0" rpy="0 0 0"/>
+            </collision> -->
             <xacro:nfr_cylinder_inertia m="0.006" r="${nfr_mini_roller_radius}" l="${nfr_mini_roller_len}" xyz="0 0 0" rpy="0 0 0"/>
         </link>

File: dev_ws/src/nfr_component_lib/urdf/nfr_odometry_pod.xacro (robot description, xacro)
@@ -24,20 +24,36 @@
             <material>Gazebo/Gray</material>
         </gazebo>
-        <link name="${link_name}_spring"/>
+        <link name="${link_name}_spring">
+            <visual>
+                <geometry>
+                    <box size="0.01 0.05 0.05"/>
+                </geometry>
+                <material name="nfr_black"/>
+                <origin xyz="0 0.025 0" rpy="0 0 0"/>
+            </visual>
+            <!-- <collision>
+                <geometry>
+                    <box size="0.011 0.043 0.043"/>
+                </geometry>
+                <origin xyz="0 0 0" rpy="0 0 0"/>
+            </collision> -->
+            <xacro:nfr_box_inertia m="0.2" x="0.01" y="0.01" z="0.01" xyz="0 0 0" rpy="0 0 0"/>
+        </link>
         <joint name="${link_name}_spring_joint" type="prismatic">
             <parent link="${link_name}"/>
+            <!-- <child link="${link_name}_mini_omni"/> -->
             <child link="${link_name}_spring"/>
             <origin xyz="0.04 0 ${-0.02-0.0205}" rpy="1.57 0 0"/>
             <axis xyz="0 1 0"/>
             <!-- max 20mm -->
-            <limit lower="0" upper="0.02" effort="1" velocity="1.0"/>
+            <limit lower="0" upper="0.02" effort="100" velocity="1"/>
             <!-- bu ne bilmiyorum -->
-            <dynamics damping="0.5" friction="0.0"/>
+            <dynamics damping="10" friction="0.1"/>
             <!-- yay sertliği değiştirilebilir -->
-            <spring_stiffness>100</spring_stiffness>
+            <spring_stiffness>10</spring_stiffness>
             <!-- yukarıdan başlat -->
-            <initial_position value="0.2"/>
+            <initial_position value="0"/>
         </joint>
-        <xacro:nfr_mini_omni_wheel link_name="${link_name}_mini_omni"/>
+        <!-- <xacro:nfr_mini_omni_wheel link_name="${link_name}_mini_omni"/>
         <joint name="${link_name}_mini_omni_joint" type="continuous">
             <parent link="${link_name}_spring"/>
@@ -45,4 +61,21 @@
             <origin xyz="0 0 0" rpy="0 0 0"/>
             <axis xyz="0 0 1"/>
+        </joint> -->
+        <link name="${link_name}_test">
+            <visual>
+                <geometry>
+                    <box size="0.03 0.03 0.01"/>
+                </geometry>
+                <material name="nfr_blue"/>
+                <origin xyz="0 0 0" rpy="0 0 0"/>
+            </visual>
+            <xacro:nfr_box_inertia m="0.1" x="0.01" y="0.01" z="0.01" xyz="0 0 0" rpy="0 0 0"/>
+        </link>
+        <joint name="${link_name}_test_joint" type="continuous">
+            <parent link="${link_name}_spring"/>
+            <child link="${link_name}_test"/>
+            <origin xyz="0 0 0" rpy="0 0 0"/>
+            <axis xyz="0 0 1"/>
+            <dynamics friction="0.1"/>
         </joint>
     </xacro:macro>

File: dev_ws/src/nfr_component_lib/urdf/nfr_omni_wheel.xacro (robot description, xacro)
@@ -30,12 +30,14 @@
             <visual>
                 <geometry>
-                    <cylinder radius="${nfr_roller_radius}" length="${nfr_roller_len}"/>
-                </geometry>
-                <material name="nfr_blue"/>
-                <origin xyz="0 0 0" rpy="0 0 0"/>
-            </visual>
-            <collision>
-                <geometry>
-                    <cylinder radius="${nfr_roller_radius}" length="${nfr_roller_len}"/>
+                    <!-- <cylinder radius="${nfr_roller_radius}" length="${nfr_roller_len}"/> -->
+                    <mesh filename="package://nfr_component_lib/meshes/mecanum_roller.stl" scale="1 1 1"/>
+                </geometry>
+                <material name="nfr_blue"/>
+                <origin xyz="0 0 0" rpy="0 0 0"/>
+            </visual>
+            <collision>
+                <geometry>
+                    <!-- <cylinder radius="${nfr_roller_radius}" length="${nfr_roller_len}"/> -->
+                    <mesh filename="package://nfr_component_lib/meshes/mecanum_roller.stl" scale="1 1 1"/>
                 </geometry>
                 <origin xyz="0 0 0" rpy="0 0 0"/>
@@ -65,12 +67,14 @@
             <visual>
                 <geometry>
-                    <cylinder radius="${nfr_roller_radius}" length="${nfr_roller_len}"/>
-                </geometry>
-                <material name="nfr_blue"/>
-                <origin xyz="0 0 0" rpy="0 0 0"/>
-            </visual>
-            <collision>
-                <geometry>
-                    <cylinder radius="${nfr_roller_radius}" length="${nfr_roller_len}"/>
+                    <!-- <cylinder radius="${nfr_roller_radius}" length="${nfr_roller_len}"/> -->
+                    <mesh filename="package://nfr_component_lib/meshes/mecanum_roller.stl" scale="1 1 1"/>
+                </geometry>
+                <material name="nfr_blue"/>
+                <origin xyz="0 0 0" rpy="0 0 0"/>
+            </visual>
+            <collision>
+                <geometry>
+                    <!-- <cylinder radius="${nfr_roller_radius}" length="${nfr_roller_len}"/> -->
+                    <mesh filename="package://nfr_component_lib/meshes/mecanum_roller.stl" scale="1 1 1"/>
                 </geometry>
                 <origin xyz="0 0 0" rpy="0 0 0"/>
@@ -100,12 +104,14 @@
             <visual>
                 <geometry>
-                    <cylinder radius="${nfr_roller_radius}" length="${nfr_roller_len}"/>
-                </geometry>
-                <material name="nfr_blue"/>
-                <origin xyz="0 0 0" rpy="0 0 0"/>
-            </visual>
-            <collision>
-                <geometry>
-                    <cylinder radius="${nfr_roller_radius}" length="${nfr_roller_len}"/>
+                    <!-- <cylinder radius="${nfr_roller_radius}" length="${nfr_roller_len}"/> -->
+                    <mesh filename="package://nfr_component_lib/meshes/mecanum_roller.stl" scale="1 1 1"/>
+                </geometry>
+                <material name="nfr_blue"/>
+                <origin xyz="0 0 0" rpy="0 0 0"/>
+            </visual>
+            <collision>
+                <geometry>
+                    <!-- <cylinder radius="${nfr_roller_radius}" length="${nfr_roller_len}"/> -->
+                    <mesh filename="package://nfr_component_lib/meshes/mecanum_roller.stl" scale="1 1 1"/>
                 </geometry>
                 <origin xyz="0 0 0" rpy="0 0 0"/>
@@ -135,12 +141,14 @@
             <visual>
                 <geometry>
-                    <cylinder radius="${nfr_roller_radius}" length="${nfr_roller_len}"/>
-                </geometry>
-                <material name="nfr_blue"/>
-                <origin xyz="0 0 0" rpy="0 0 0"/>
-            </visual>
-            <collision>
-                <geometry>
-                    <cylinder radius="${nfr_roller_radius}" length="${nfr_roller_len}"/>
+                    <!-- <cylinder radius="${nfr_roller_radius}" length="${nfr_roller_len}"/> -->
+                    <mesh filename="package://nfr_component_lib/meshes/mecanum_roller.stl" scale="1 1 1"/>
+                </geometry>
+                <material name="nfr_blue"/>
+                <origin xyz="0 0 0" rpy="0 0 0"/>
+            </visual>
+            <collision>
+                <geometry>
+                    <!-- <cylinder radius="${nfr_roller_radius}" length="${nfr_roller_len}"/> -->
+                    <mesh filename="package://nfr_component_lib/meshes/mecanum_roller.stl" scale="1 1 1"/>
                 </geometry>
                 <origin xyz="0 0 0" rpy="0 0 0"/>
@@ -170,12 +178,14 @@
             <visual>
                 <geometry>
-                    <cylinder radius="${nfr_roller_radius}" length="${nfr_roller_len}"/>
-                </geometry>
-                <material name="nfr_blue"/>
-                <origin xyz="0 0 0" rpy="0 0 0"/>
-            </visual>
-            <collision>
-                <geometry>
-                    <cylinder radius="${nfr_roller_radius}" length="${nfr_roller_len}"/>
+                    <!-- <cylinder radius="${nfr_roller_radius}" length="${nfr_roller_len}"/> -->
+                    <mesh filename="package://nfr_component_lib/meshes/mecanum_roller.stl" scale="1 1 1"/>
+                </geometry>
+                <material name="nfr_blue"/>
+                <origin xyz="0 0 0" rpy="0 0 0"/>
+            </visual>
+            <collision>
+                <geometry>
+                    <!-- <cylinder radius="${nfr_roller_radius}" length="${nfr_roller_len}"/> -->
+                    <mesh filename="package://nfr_component_lib/meshes/mecanum_roller.stl" scale="1 1 1"/>
                 </geometry>
                 <origin xyz="0 0 0" rpy="0 0 0"/>
@@ -205,12 +215,14 @@
             <visual>
                 <geometry>
-                    <cylinder radius="${nfr_roller_radius}" length="${nfr_roller_len}"/>
-                </geometry>
-                <material name="nfr_blue"/>
-                <origin xyz="0 0 0" rpy="0 0 0"/>
-            </visual>
-            <collision>
-                <geometry>
-                    <cylinder radius="${nfr_roller_radius}" length="${nfr_roller_len}"/>
+                    <!-- <cylinder radius="${nfr_roller_radius}" length="${nfr_roller_len}"/> -->
+                    <mesh filename="package://nfr_component_lib/meshes/mecanum_roller.stl" scale="1 1 1"/>
+                </geometry>
+                <material name="nfr_blue"/>
+                <origin xyz="0 0 0" rpy="0 0 0"/>
+            </visual>
+            <collision>
+                <geometry>
+                    <!-- <cylinder radius="${nfr_roller_radius}" length="${nfr_roller_len}"/> -->
+                    <mesh filename="package://nfr_component_lib/meshes/mecanum_roller.stl" scale="1 1 1"/>
                 </geometry>
                 <origin xyz="0 0 0" rpy="0 0 0"/>
@@ -240,12 +252,14 @@
             <visual>
                 <geometry>
-                    <cylinder radius="${nfr_roller_radius}" length="${nfr_roller_len}"/>
-                </geometry>
-                <material name="nfr_blue"/>
-                <origin xyz="0 0 0" rpy="0 0 0"/>
-            </visual>
-            <collision>
-                <geometry>
-                    <cylinder radius="${nfr_roller_radius}" length="${nfr_roller_len}"/>
+                    <!-- <cylinder radius="${nfr_roller_radius}" length="${nfr_roller_len}"/> -->
+                    <mesh filename="package://nfr_component_lib/meshes/mecanum_roller.stl" scale="1 1 1"/>
+                </geometry>
+                <material name="nfr_blue"/>
+                <origin xyz="0 0 0" rpy="0 0 0"/>
+            </visual>
+            <collision>
+                <geometry>
+                    <!-- <cylinder radius="${nfr_roller_radius}" length="${nfr_roller_len}"/> -->
+                    <mesh filename="package://nfr_component_lib/meshes/mecanum_roller.stl" scale="1 1 1"/>
                 </geometry>
                 <origin xyz="0 0 0" rpy="0 0 0"/>
@@ -275,12 +289,14 @@
             <visual>
                 <geometry>
-                    <cylinder radius="${nfr_roller_radius}" length="${nfr_roller_len}"/>
-                </geometry>
-                <material name="nfr_blue"/>
-                <origin xyz="0 0 0" rpy="0 0 0"/>
-            </visual>
-            <collision>
-                <geometry>
-                    <cylinder radius="${nfr_roller_radius}" length="${nfr_roller_len}"/>
+                    <!-- <cylinder radius="${nfr_roller_radius}" length="${nfr_roller_len}"/> -->
+                    <mesh filename="package://nfr_component_lib/meshes/mecanum_roller.stl" scale="1 1 1"/>
+                </geometry>
+                <material name="nfr_blue"/>
+                <origin xyz="0 0 0" rpy="0 0 0"/>
+            </visual>
+            <collision>
+                <geometry>
+                    <!-- <cylinder radius="${nfr_roller_radius}" length="${nfr_roller_len}"/> -->
+                    <mesh filename="package://nfr_component_lib/meshes/mecanum_roller.stl" scale="1 1 1"/>
                 </geometry>
                 <origin xyz="0 0 0" rpy="0 0 0"/>
@@ -310,12 +326,14 @@
             <visual>
                 <geometry>
-                    <cylinder radius="${nfr_roller_radius}" length="${nfr_roller_len}"/>
-                </geometry>
-                <material name="nfr_blue"/>
-                <origin xyz="0 0 0" rpy="0 0 0"/>
-            </visual>
-            <collision>
-                <geometry>
-                    <cylinder radius="${nfr_roller_radius}" length="${nfr_roller_len}"/>
+                    <!-- <cylinder radius="${nfr_roller_radius}" length="${nfr_roller_len}"/> -->
+                    <mesh filename="package://nfr_component_lib/meshes/mecanum_roller.stl" scale="1 1 1"/>
+                </geometry>
+                <material name="nfr_blue"/>
+                <origin xyz="0 0 0" rpy="0 0 0"/>
+            </visual>
+            <collision>
+                <geometry>
+                    <!-- <cylinder radius="${nfr_roller_radius}" length="${nfr_roller_len}"/> -->
+                    <mesh filename="package://nfr_component_lib/meshes/mecanum_roller.stl" scale="1 1 1"/>
                 </geometry>
                 <origin xyz="0 0 0" rpy="0 0 0"/>
@@ -345,12 +363,14 @@
             <visual>
                 <geometry>
-                    <cylinder radius="${nfr_roller_radius}" length="${nfr_roller_len}"/>
-                </geometry>
-                <material name="nfr_blue"/>
-                <origin xyz="0 0 0" rpy="0 0 0"/>
-            </visual>
-            <collision>
-                <geometry>
-                    <cylinder radius="${nfr_roller_radius}" length="${nfr_roller_len}"/>
+                    <!-- <cylinder radius="${nfr_roller_radius}" length="${nfr_roller_len}"/> -->
+                    <mesh filename="package://nfr_component_lib/meshes/mecanum_roller.stl" scale="1 1 1"/>
+                </geometry>
+                <material name="nfr_blue"/>
+                <origin xyz="0 0 0" rpy="0 0 0"/>
+            </visual>
+            <collision>
+                <geometry>
+                    <!-- <cylinder radius="${nfr_roller_radius}" length="${nfr_roller_len}"/> -->
+                    <mesh filename="package://nfr_component_lib/meshes/mecanum_roller.stl" scale="1 1 1"/>
                 </geometry>
                 <origin xyz="0 0 0" rpy="0 0 0"/>
@@ -380,12 +400,14 @@
             <visual>
                 <geometry>
-                    <cylinder radius="${nfr_roller_radius}" length="${nfr_roller_len}"/>
-                </geometry>
-                <material name="nfr_blue"/>
-                <origin xyz="0 0 0" rpy="0 0 0"/>
-            </visual>
-            <collision>
-                <geometry>
-                    <cylinder radius="${nfr_roller_radius}" length="${nfr_roller_len}"/>
+                    <!-- <cylinder radius="${nfr_roller_radius}" length="${nfr_roller_len}"/> -->
+                    <mesh filename="package://nfr_component_lib/meshes/mecanum_roller.stl" scale="1 1 1"/>
+                </geometry>
+                <material name="nfr_blue"/>
+                <origin xyz="0 0 0" rpy="0 0 0"/>
+            </visual>
+            <collision>
+                <geometry>
+                    <!-- <cylinder radius="${nfr_roller_radius}" length="${nfr_roller_len}"/> -->
+                    <mesh filename="package://nfr_component_lib/meshes/mecanum_roller.stl" scale="1 1 1"/>
                 </geometry>
                 <origin xyz="0 0 0" rpy="0 0 0"/>
@@ -415,12 +437,14 @@
             <visual>
                 <geometry>
-                    <cylinder radius="${nfr_roller_radius}" length="${nfr_roller_len}"/>
-                </geometry>
-                <material name="nfr_blue"/>
-                <origin xyz="0 0 0" rpy="0 0 0"/>
-            </visual>
-            <collision>
-                <geometry>
-                    <cylinder radius="${nfr_roller_radius}" length="${nfr_roller_len}"/>
+                    <!-- <cylinder radius="${nfr_roller_radius}" length="${nfr_roller_len}"/> -->
+                    <mesh filename="package://nfr_component_lib/meshes/mecanum_roller.stl" scale="1 1 1"/>
+                </geometry>
+                <material name="nfr_blue"/>
+                <origin xyz="0 0 0" rpy="0 0 0"/>
+            </visual>
+            <collision>
+                <geometry>
+                    <!-- <cylinder radius="${nfr_roller_radius}" length="${nfr_roller_len}"/> -->
+                    <mesh filename="package://nfr_component_lib/meshes/mecanum_roller.stl" scale="1 1 1"/>
                 </geometry>
                 <origin xyz="0 0 0" rpy="0 0 0"/>

File: dev_ws/src/nfr_component_lib/urdf/nfr_structure.xacro (robot description, xacro)
@@ -5,6 +5,6 @@
         <!-- boş olan taraf üste (+z) bakıyor -->
         <!-- şimdilik böyle yapıyorum affedin beni -->
-        <!-- <xacro:nfr_box_inertia m="${step*0.020}" x="${step*0.025}" y="0.05" z="0.05" xyz="${xyz}" rpy="${rpy}"/> -->
-        <xacro:nfr_box_inertia m="0.0001" x="${step*0.025}" y="0.05" z="0.05" xyz="${xyz}" rpy="${rpy}"/>
+        <xacro:nfr_box_inertia m="${step*0.020}" x="${step*0.025}" y="0.05" z="0.05" xyz="${xyz}" rpy="${rpy}"/>
+        <!-- <xacro:nfr_box_inertia m="0.0001" x="${step*0.025}" y="0.05" z="0.05" xyz="${xyz}" rpy="${rpy}"/> -->
     </xacro:macro>
     <xacro:macro name="nfr_structure" params="link_name step xyz rpy">
